Commit message: Gazebo

File: washer_description/urdf/robot.urdf (robot description, URDF)
Before this commit: robot washer_robot, 5 links, 4 joints
Links:
- added link base_footprint
- link lidar_link: mass None -> 0.1
Joints:
- added joint base_footprint_joint: type fixed, parent base_footprint, child base_link, origin xyz=0 0 0.4 rpy=0 0 0
- joint caster_wheel_joint: origin xyz=0.35 0 0.06 rpy=0 0 0 -> xyz=0.35 0 -0.34 rpy=0 0 0
- joint lidar_joint: origin xyz=0.1 0 0.63 rpy=0 0 0 -> xyz=0.1 0 0.4 rpy=0 0 0
- joint rear_left_wheel_joint: origin xyz=-0.3 0.32 0.12 rpy=0 0 0 -> xyz=-0.3 0.28 -0.28 rpy=0 0 0
- joint rear_right_wheel_joint: origin xyz=-0.3 -0.32 0.12 rpy=0 0 0 -> xyz=-0.3 -0.28 -0.28 rpy=0 0 0
