Commit message: temp

File: src/washer_description/urdf/robot.urdf (robot description, URDF)
Before this commit: robot washer_robot, 6 links, 5 joints
Links:
- link base_link: mass 50.0 -> 5.0
- link caster_wheel: mass 0.5 -> None; geometry visual sphere radius=0.06
Joints:
- joint base_footprint_joint: origin xyz=0 0 0.4 rpy=0 0 0 -> xyz=0 0 0.25 rpy=0 0 0
- joint caster_wheel_joint: origin xyz=0.35 0 -0.34 rpy=0 0 0 -> xyz=0.35 0 -0.19 rpy=0 0 0
- joint rear_left_wheel_joint: origin xyz=-0.3 0.28 -0.28 rpy=0 0 0 -> xyz=-0.3 0.28 -0.13 rpy=0 0 0
- joint rear_right_wheel_joint: origin xyz=-0.3 -0.28 -0.28 rpy=0 0 0 -> xyz=-0.3 -0.28 -0.13 rpy=0 0 0

Commit message: Fix: visualization LIDAR, UPD: README

File: src/washer_description/urdf/robot.urdf (robot description, URDF)
Before this commit: robot washer_robot, 6 links, 5 joints
Links:
- link base_link: mass 5.0 -> 40.0
- link caster_wheel: mass None -> 0.01; geometry collision sphere radius=0.06; visual sphere radius=0.06
Joints:
- joint base_footprint_joint: origin xyz=0 0 0.25 rpy=0 0 0 -> xyz=0 0 0.35 rpy=0 0 0
- joint lidar_joint: origin xyz=0.1 0 0.4 rpy=0 0 0 -> xyz=0.1 0 0.52 rpy=0 0 0
